File: plc/kicad/LibrePLC32.kicad_pcb (KiCad board)
At the start: 2 copper layers, 228 parts, among them CN1 DB128V-5.08-2P-GN-S, CN10 DB2ERC-5.08-4P, CN11 DB2ERC-5.08-4P, CN2 DB128V-5.08-2P-GN-S, CN3 DB128V-5.08-2P-GN-S, CN4 DB128V-5.08-2P-GN-S, CN5 DB128V-5.08-2P-GN-S, CN6 DB128V-5.08-2P-GN-S, CN7 DB128V-5.08-2P-GN-S, CN8 DB128V-5.08-2P-GN-S, CN9 DB128V-5.08-6P-GN-S, Q1 AO3400A, Q2 AO3400A, Q3 L8050QLT1G, Q4 L8050QLT1G, Q5 BSS138LT1G, Q6 CSD19537Q3, SW1 TSD003B08026A03, SW2 TSD003B08026A03, SW3 TSD003B08026A03, SW4 MSK12C02, SW5 MSK12C02, U1 TCA9535PWR, U10 CP2102N-A02-GQFN28R, U11 LMR16006XDDCR, U12 TPS54560DDAR, U13 TPS26630RGER, U14 TCAN337DR, U15 THVD1450DR, U16 W5500, U17 TLV76733DRVR, U2 TPS272C45DRHFR, U3 TPS272C45DRHFR, U4 ADS1115IDGSR, U5 LTV-814S-TA1-A, U6 LTV-814S-TA1-A, U7 LTV-814S-TA1-A, U8 LTV-814S-TA1-A, U9 ESP32-S3-MINI-1U, X1 X322525MRB4SI

Commit message: PCB placement
Parts:
- added C12: 100n, Capacitor_SMD:C_0603_1608Metric, F.Cu at (367.7, 22.2)
- added C13: 100n, Capacitor_SMD:C_0603_1608Metric, F.Cu at (367.7, 25.7)
- added C15: 100n, Capacitor_SMD:C_0603_1608Metric, F.Cu at (235.9, 115.5)
- added C21: 220u, Capacitor_SMD:C_0603_1608Metric, F.Cu at (241.5, 136.8)
- added CN2: DB128V-5.08-2P-GN-S, LibrePLC32:CONN-TH_2P-P5.08_DIBO_DB128V-5.08, F.Cu at (-91.9, 105.7)
- added J2: Conn_01x04_Pin, Connector_PinSocket_2.54mm:PinSocket_1x04_P2.54mm_Vertical, F.Cu at (231.6, 111.5)
- added R44: 5.1k, Resistor_SMD:R_0603_1608Metric, F.Cu at (373.7, 25.7)
- added TP10: TestPoint, TestPoint:TestPoint_Pad_D3.0mm, F.Cu at (-103.0, -45.5)
- added TP17: TestPoint, TestPoint:TestPoint_Pad_D3.0mm, F.Cu at (-34.5, -52.0)
- added TP18: TestPoint, TestPoint:TestPoint_Pad_D3.0mm, F.Cu at (-44.5, -43.0)
- added TP19: TestPoint, TestPoint:TestPoint_Pad_D3.0mm, F.Cu at (426.5, 343.0)
- added TP20: TestPoint, TestPoint:TestPoint_Pad_D3.0mm, F.Cu at (413.5, 343.0)
- added TP21: TestPoint, TestPoint:TestPoint_Pad_D3.0mm, F.Cu at (231.9, 138.1)
- added TP22: TestPoint, TestPoint:TestPoint_Pad_D3.0mm, F.Cu at (231.9, 143.1)
- added TP23: TestPoint, TestPoint:TestPoint_Pad_D3.0mm, F.Cu at (236.9, 138.1)
- added TP24: TestPoint, TestPoint:TestPoint_Pad_D4.0mm, F.Cu at (227.3, 126.5)
- added TP25: TestPoint, TestPoint:TestPoint_Pad_D4.0mm, F.Cu at (227.3, 132.5)
- added TP26: TestPoint, TestPoint:TestPoint_Pad_D4.0mm, F.Cu at (233.4, 126.5)
- added TP27: TestPoint, TestPoint:TestPoint_Pad_D4.0mm, F.Cu at (233.4, 132.5)
- added TP28: TestPoint, TestPoint:TestPoint_Pad_D3.0mm, F.Cu at (236.9, 143.1)
- added TP29: TestPoint, TestPoint:TestPoint_Pad_D4.0mm, F.Cu at (239.4, 126.5)
- added TP30: TestPoint, TestPoint:TestPoint_Pad_D4.0mm, F.Cu at (239.4, 132.5)
- added TP31: TestPoint, TestPoint:TestPoint_Pad_D4.0mm, F.Cu at (245.5, 126.5)
- added TP32: TestPoint, TestPoint:TestPoint_Pad_D4.0mm, F.Cu at (245.5, 132.5)
- added TP9: TestPoint, TestPoint:TestPoint_Pad_D3.0mm, F.Cu at (-92.5, -54.5)
- added U11: BS-0601-SK-4W, LibrePLC32:BAT-SMD_BS-06-B4AA012, F.Cu at (369.7, 10.5)
- added U12: AHT20_C2757850, LibrePLC32:SENSOR-SMD_L3.0-W3.0-P1.00-BR, F.Cu at (240.0, 111.3)
- added U9: RV-3028-C7, LibrePLC32:OSC-SMD_8P-L3.2-W1.5-P0.90-BL, F.Cu at (370.3, 24.1)
- C18: renamed from C15; value 47u -> 220u
- TP1, TP12, TP2, TP3, TP4, TP5, TP6, TP7, TP8: footprint TestPoint:TestPoint_Pad_D3.0mm -> TestPoint:TestPoint_Pad_D2.0mm
- TP11: renamed from TP9; footprint TestPoint:TestPoint_Pad_D3.0mm -> TestPoint:TestPoint_Pad_D2.0mm
- TP13: renamed from TP11; footprint TestPoint:TestPoint_Pad_D3.0mm -> TestPoint:TestPoint_Pad_D2.0mm
- TP14: renamed from TP10; footprint TestPoint:TestPoint_Pad_D3.0mm -> TestPoint:TestPoint_Pad_D2.0mm
- TP15: renamed from TP13; footprint TestPoint:TestPoint_Pad_D3.0mm -> TestPoint:TestPoint_Pad_D2.0mm
- TP16: renamed from TP14; footprint TestPoint:TestPoint_Pad_D3.0mm -> TestPoint:TestPoint_Pad_D2.0mm
- moved U8 362.5 mm to (-200.5, 86.5)
- moved U7 346.1 mm to (-190.5, 86.5)
- moved R69 343.7 mm to (418.0, 343.0), turned to 180 degrees
- moved R39 340.4 mm to (-202.5, 78.0), turned to -90 degrees
- moved D7 336.7 mm to (421.9, 343.0)
- moved R35 334.5 mm to (-197.0, 80.7), turned to -90 degrees
- moved CN9 334.4 mm to (-200.8, 102.0)
- moved R27 334.0 mm to (-200.5, 96.0), turned to 180 degrees
- moved R31 330.1 mm to (-196.5, 95.0), turned to 90 degrees
- moved R38 329.8 mm to (-192.0, 78.0), turned to -90 degrees
- moved U6 329.6 mm to (-180.3, 86.5)
- moved D3 329.0 mm to (-147.0, 200.0), turned to -90 degrees
- moved C28 327.3 mm to (383.7, 338.0)
- moved C31 327.3 mm to (383.7, 345.5)
- moved R59 327.3 mm to (387.7, 345.5)
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- renumbered C12 to C14, C13 to C16, C14 to C17, C16 to C19, C17 to C20, C19 to C22, C20 to C23, C21 to C24, C18 to C25, C22 to C26, C23 to C27, C24 to C28, C25 to C29, C26 to C30, C27 to C31, C28 to C32, C29 to C33, C30 to C34, C31 to C35, C32 to C36, C48 to C37, C50 to C38, C49 to C39, C33 to C40, C34 to C41, C35 to C42, C36 to C43, C37 to C44, C38 to C45, C39 to C46, C40 to C47, C41 to C48, C42 to C49, C43 to C50, C44 to C51, C45 to C52, C46 to C53, C47 to C54, CN9 to CN10, CN10 to CN11, CN11 to CN12, CN6 to CN3, CN7 to CN4, CN8 to CN5, CN2 to CN6, CN3 to CN7, CN4 to CN8, CN5 to CN9, D15 to D10, D17 to D11, D9 to D12, D10 to D13, D16 to D14, D11 to D15, D12 to D16, D13 to D17, D14 to D18, D18 to D9, F6 to F3, F7 to F4, F4 to F5, F5 to F6, R44 to R45, R45 to R46, R46 to R47, R47 to R48, R50 to R49, R51 to R50, R52 to R51, R53 to R52, R54 to R53, R55 to R54, R56 to R55, R57 to R56, R48 to R57, R49 to R58, R58 to R59, R59 to R60, R60 to R61, R61 to R62, R62 to R63, R63 to R64, R64 to R65, R65 to R66, R66 to R67, R67 to R68, R68 to R69, R69 to R70, R70 to R71, R71 to R72, R72 to R73, R92 to R74, R73 to R75, R74 to R76, R75 to R77, R76 to R78, R91 to R79, R77 to R80, R78 to R81, R79 to R82, R80 to R83, R81 to R84, R82 to R85, R83 to R86, R84 to R87, R85 to R88, R86 to R89, R87 to R90, R88 to R91, R89 to R92, R90 to R93, U9 to U10, U10 to U13, U11 to U14, U12 to U15, U13 to U16, U14 to U18, U15 to U19, U16 to U20
Connections:
- net Net-(U9-IO4) renamed /MCU/~{RTC_INT}
- CN11 pad 3: /CAN/CAN_L -> /CAN/CAN_H
- CN11 pad 4: /CAN/CAN_H -> /CAN/CAN_L
- U19 pad 8: unconnected-(U15-VCC-Pad8) -> +3V3
Other:
- copper layers 2 -> 4
