File: plc/kicad/LibrePLC32.kicad_pcb (KiCad board)
At the start: 4 copper layers, 154.5 x 112.9 mm, 295 parts, among them CN1 DB128V-5.08-2P-GN-S, CN10 DB128V-5.08-2P-GN-S, CN11 DB2ERC-5.08-4P, CN12 DB2ERC-5.08-4P, CN13 DB128V-5.08-2P-GN-S, CN14 DB128V-5.08-2P-GN-S, CN2 DB128V-5.08-2P-GN-S, CN3 DB128V-5.08-2P-GN-S, CN4 DB128V-5.08-2P-GN-S, CN5 DB128V-5.08-2P-GN-S, CN6 DB128V-5.08-2P-GN-S, CN7 DB128V-5.08-2P-GN-S, CN8 DB128V-5.08-2P-GN-S, CN9 DB128V-5.08-2P-GN-S, J2 Conn_01x04_Pin, J3 Conn_01x02_Pin, Q1 AO3400A, Q2 AO3400A, Q3 L8050QLT1G, Q4 L8050QLT1G, Q5 BSS138LT1G, Q6 CSD19537Q3, SW1 TSD003B08026A03, SW2 TSD003B08026A03, SW3 TSD003B08026A03, SW4 MSK12C02, SW5 MSK12C02, U1 TCA9535PWR, U10 ESP32-S3-MINI-1U, U11 BS-0601-SK-4W, U12 AHT20_C2757850, U13 CP2102N-A02-GQFN28R, U14 ISO1042BDWVR, U15 TPS54560BDDAR, U16 TPS26630RGER, U17 TPS7A5201QRGRRQ1, U18 ISO1500DBQR, U2 TPS272C45DRHFR, U20 W5500, U21 BZT52C3V3S, U22 B0505XT-1WR3, U23 B0505XT-1WR3, U3 TPS272C45DRHFR, U4 ADS1115IDGSR, U5 LTV-814S-TA1-A, U6 LTV-814S-TA1-A, U7 LTV-814S-TA1-A, U8 LTV-814S-TA1-A, U9 RV-3028-C7, X1 X322525MRB4SI

Commit message: Added i2c addresses & TPS26630 modifications
Changed lines of the file:
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@@
 		(tags "resistor")
 		(property "Reference" "R101"
-			(at -3.075 0 0)
+			(at -3.260345 0 0)
 			(layer "F.SilkS")
-			(hide yes)
 			(effects
 				(font

Commit message: Needed fixes
Parts:
- R85: value 73.2k -> 100k
- U12: value AHT20_C2757850 -> AHT20
Routing:
- net GND: vias 337 -> 336
Changed lines of the file:
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@@
 			)
 		)
-		(property "Value" "AHT20_C2757850"
+		(property "Value" "AHT20"
 			(at 0 5 0)
 			(layer "F.Fab")
@@
 			)
 		)
-		(property "Value" "73.2k"
+		(property "Value" "100k"
 			(at 0 1.43 0)
 			(layer "F.Fab")
@@
 		(size 0.5)
 		(drill 0.3)
-		(layers "F.Cu" "B.Cu")
-		(net "GND")
-	)
-	(via
-		(at 104.879655 55.212857)
-		(size 0.5)
-		(drill 0.3)
