File: plc/kicad/power.kicad_sch (KiCad schematic)
At the start: 82 parts, among them Q5 BSS138LT1G, Q6 CSD19537Q3, SW3 TSD003B08026A03, U15 TPS54560BDDAR, U16 TPS26630RGER, U17 TPS7A5201QRGRRQ1, U21 BZT52C3V3S

Commit message: Added i2c addresses & TPS26630 modifications
Other:
- note added: "TO FIX MODE TO FLOATING!!"
Changed lines of the file:
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@@
 		)
 	)
+	(text "TO FIX MODE TO FLOATING!!"
+		(exclude_from_sim no)
+		(at 130.81 194.31 0)
+		(effects
+			(font
+				(size 3 3)
+				(thickness 0.6)
+				(bold yes)
+			)
+		)
+	)
 	(text "1%"
 		(exclude_from_sim no)
@@
 		(dnp no)
 		(property "Reference" "D14"
-			(at 310.515 233.68 0)
+			(at 311.15 242.57 0)
 			(show_name no)
 			(do_not_autoplace no)
